File: SmaCon.kicad_pcb (KiCad board)
At the start: 2 copper layers, 0 parts

Commit message: 基板 V1.0
Parts:
- added 1: , clipboard:22b1b73a-550e-4fe2-9098-770367972fd8, F.Cu at (0.00, 68.5)
- added 2: , clipboard:22b1b73a-550e-4fe2-9098-770367972fd8, F.Cu at (-17.0, 68.1)
- added C1: 2.2uF, SmaCon:1005Metric, F.Cu at (15.0, 51.7)
- added C10: 2.2uF, SmaCon:1005Metric, F.Cu at (-2.70, 18.9)
- added C11: 0.1uF, SmaCon:1005Metric, F.Cu at (9.00, 28.8)
- added C12: 10uF, SmaCon:1608Metric, F.Cu at (-12.0, 45.2)
- added C13: 1uF, SmaCon:1005Metric, F.Cu at (-8.75, 28.9)
- added C14: 4.7uF, SmaCon:1608Metric, F.Cu at (-20.0, 59.0)
- added C15: 10pF, SmaCon:1005Metric, F.Cu at (-15.5, 60.0)
- added C16: 10pF, SmaCon:1005Metric, F.Cu at (-15.5, 55.0)
- added C17: 10uF, SmaCon:1608Metric, F.Cu at (1.10, 45.0)
- added C2: 2.2uF, SmaCon:1005Metric, F.Cu at (17.0, 51.7)
- added C3: 10uF, SmaCon:1608Metric, F.Cu at (19.4, 52.9)
- added C4: 0.1uF, SmaCon:1005Metric, F.Cu at (16.5, 42.0)
- added C5: 10uF, SmaCon:1608Metric, F.Cu at (-10.3, 29.5)
- added C6: 0.1uF, SmaCon:1005Metric, F.Cu at (-5.20, 18.9)
- added C7: 0.1uF, SmaCon:1005Metric, F.Cu at (-20.0, 63.2)
- added C8: 0.1uF, SmaCon:1005Metric, F.Cu at (4.85, 38.2)
- added C9: 2.2uF, SmaCon:1005Metric, F.Cu at (4.85, 39.5)
- added F1: Polyfuse, SmaCon:3216Metric, F.Cu at (10.0, 62.0)
- added J1: USB_C_Receptacle, SmaCon:USB Type-C 5077CR-16SMC2-BK-TR, F.Cu at (0.00, 92.6)
- added J2: ST7789, SmaCon:Hirose_FH12-18S-0.5SH_1x18-1MP_P0.50mm_Horizontal, B.Cu at (0.00, 19.0)
- added J3: GT911, SmaCon:Hirose_FH12-6S-0.5SH_1x06-1MP_P0.50mm_Horizontal, B.Cu at (-17.0, 39.0)
- added J4: AudioJack, SmaCon:PJ-3420, F.Cu at (-16.5, 0.00)
- added J5: STM32_Debug, SmaCon:STM32_Debug_5pin, F.Cu at (-4.20, 38.9)
- added J6: Conn_01x04, SmaCon:PinHeader_1x04_P2.54mm_Horizontal, F.Cu at (13.2, 12.2)
- added L1: L, SmaCon:1608Metric, F.Cu at (10.0, 55.0)
- added L2: 2.2uH, SmaCon:2012Metric, F.Cu at (-0.80, 19.7)
- added LS1: Speaker, SmaCon:micro_speaker, F.Cu at (0.00, 81.0)
- added M1: LD14-002, SmaCon:LD14-002, F.Cu at (0.00, 57.5)
- added Q1: AO3400A, SmaCon:SOT-23, F.Cu at (2.20, 17.4)
- added R1: 5.1k, SmaCon:1005Metric, F.Cu at (17.0, 63.5)
- added R10: 100, SmaCon:2012Metric, F.Cu at (-20.5, 29.3)
- added R11: 100, SmaCon:2012Metric, F.Cu at (-17.5, 29.3)
- added R12: 10k, SmaCon:1005Metric, F.Cu at (-3.00, 11.0)
- added R13: 4.7k, SmaCon:1005Metric, F.Cu at (0.00, 11.0)
- added R14: 10k, SmaCon:1005Metric, F.Cu at (3.00, 11.0)
- added R15: 10k, SmaCon:1005Metric, F.Cu at (10.4, 42.0)
- added R2: 5.1k, SmaCon:1005Metric, F.Cu at (13.0, 63.5)
- added R3: 10k, SmaCon:1005Metric, F.Cu at (13.5, 42.0)
- added R4: 470, SmaCon:1005Metric, F.Cu at (1.25, 20.6)
- added R5: 10k, SmaCon:1005Metric, F.Cu at (3.15, 20.6)
- added R6: 100, SmaCon:2012Metric, F.Cu at (-14.5, 29.3)
- added R7: 100, SmaCon:2012Metric, F.Cu at (-12.3, 29.3)
- added R8: 10k, SmaCon:1005Metric, F.Cu at (-20.0, 55.0)
- added R9: 1M, SmaCon:1005Metric, F.Cu at (-15.5, 57.5)
- added RV1: Potentiometer_Dual, SmaCon:JT8P-3.2T-B10K-1-16Y, F.Cu at (-19.0, 80.0)
- added SW1: SW_Push, SmaCon:tact_switch, F.Cu at (25.0, 80.0)
- added SW2: SW_Push, SmaCon:tact_switch, F.Cu at (18.0, 87.0)
- added SW3: SW_Push, SmaCon:tact_switch, F.Cu at (11.0, 80.0)
- added SW4: SW_Push, SmaCon:tact_switch, F.Cu at (18.0, 73.0)
- added SW5: SW_TMHU27, SmaCon:SW_TMHU27, F.Cu at (0.00, 4.00)
- added TP1: TestPoint, SmaCon:TestPoint_THTPad_D1.2mm_Drill0.8mm, F.Cu at (9.00, 34.0)
- added U1: LXES11DAA2-137, SmaCon:LXES11D, F.Cu at (15.0, 63.5)
- added U2: NJM2884U1, SmaCon:SOT-89-5, F.Cu at (16.0, 56.0)
- added U3: BD45285, SmaCon:SOT-23-5, F.Cu at (15.0, 45.0)
- added U4: STM32U575CIUxQ, SmaCon:QFN-48-1EP_7x7mm_P0.5mm_EP5.3x5.3mm, F.Cu at (0.00, 30.0)
- added U5: YMF825, SmaCon:SSOP-24_5.3x8.2mm_P0.65mm, F.Cu at (-18.0, 45.1)
- added U6: 25LC080C, SmaCon:MSOP-8_3x3mm_P0.65mm, F.Cu at (7.05, 45.0)
- added U7: BD6211, SmaCon:SOP-8_4.4x5.0mm_P1.27mm, F.Cu at (-4.42, 45.0)
- added Y1: 12.288MHz, SmaCon:Crystal_SMD_TXC_AX_8045-2Pin_8.0x4.5mm, F.Cu at (-12.0, 57.5)
Routing:
- net +3.3V: track 0.00 -> 253.2 mm, vias 0 -> 10
- net POS_H: track 0.00 -> 110.9 mm, vias 0 -> 1
- net POS_V: track 0.00 -> 96.8 mm, vias 0 -> 1
- net GND: track 0.00 -> 93.1 mm, vias 0 -> 116
- net SW_B: track 0.00 -> 88.3 mm, vias 0 -> 1
- net RESET: track 0.00 -> 79.8 mm, vias 0 -> 4
- net SW_C: track 0.00 -> 75.9 mm, vias 0 -> 1
- net +5V: track 0.00 -> 73.2 mm
- net SW_A: track 0.00 -> 64.8 mm
- net SW_D: track 0.00 -> 62.7 mm, vias 0 -> 1
- net AUDIO_SW: track 0.00 -> 58.3 mm, vias 0 -> 2
- net USB_DM: track 0.00 -> 57.2 mm, vias 0 -> 2
- net USB_DP: track 0.00 -> 54.8 mm, vias 0 -> 2
- net Net-(U5-SPOUT1): track 0.00 -> 41.7 mm
- net Net-(F1-Pad2): track 0.00 -> 40.4 mm, vias 0 -> 2
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- added copper zone on B.Cu, net GND
- added copper zone on F.Cu, net GND
Other:
- board outline added: 60 x 100 mm
- board text added: "SmaCon"
- board text added: "V1.0"

Commit message: 基板 V1.1
Parts:
- moved J2 2.60 mm to (0.00, 21.6)
- moved TP1 2.10 mm to (6.90, 34.0)
- moved J3 1.85 mm to (-17.0, 40.9)
Connections:
- RV1 pad 2: POS_H -> POS_V
- RV1 pad 5: POS_V -> POS_H
Routing:
- net GND: track 93.1 -> 111.4 mm, vias 116 -> 121
- net POS_H: track 110.9 -> 96.4 mm
- net POS_V: track 96.8 -> 109.2 mm
- net +3.3V: track 253.2 -> 264.4 mm
- net TFT_CS: track 19.3 -> 13.3 mm, vias 1 -> 3
- net Net-(Q1-D): track 10.4 -> 7.67 mm
- net TFT_CLK: track 10.0 -> 12.4 mm
- net /TEST: track 6.27 -> 4.17 mm
- net Net-(J2-LEDA): track 28.5 -> 30.5 mm
- net AUDIO_SW: track 58.3 -> 56.7 mm
- net MOTOR_RIN: track 33.0 -> 34.4 mm
- net TFT_DC: track 10.0 -> 11.1 mm
- net RESET: track 79.8 -> 80.6 mm
- net MOTOR_FIN: track 23.6 -> 24.3 mm
- net SW_D: track 62.7 -> 63.3 mm
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Other:
- board text added: "V1.1"
- board text removed: "V1.0"

Commit message: 基板 V1.2
Routing:
- net GND: track 111.4 -> 145.0 mm, vias 121 -> 126
- net TFT_CLK: track 12.4 -> 14.5 mm
- net TFT_MOSI: track 10.3 -> 12.4 mm
- net SOUND_CLK: track 20.8 -> 22.5 mm
- net RESET: track 80.6 -> 82.0 mm
- net SOUND_MISO: track 19.6 -> 20.7 mm
- net SOUND_MOSI: track 23.4 -> 24.3 mm
- net LEVER_SW: track 31.8 -> 32.5 mm
- net TFT_DC: track 11.1 -> 11.6 mm
Other:
- board text added: "V1.2"
- board text removed: "V1.1"

Commit message: 基板 V2.0
Parts:
- added R16: 50, SmaCon:1005Metric, F.Cu at (3.00, 24.3)
- added R17: 50, SmaCon:1005Metric, F.Cu at (2.00, 24.3)
- added R18: 50, SmaCon:1005Metric, F.Cu at (1.00, 24.3)
- moved J4 16.6 mm to (0.05, 0.03)
- moved SW5 15.1 mm to (-15.0, 6.00)
- moved R12 15.0 mm to (-17.9, 12.7)
- moved R13 15.0 mm to (-14.9, 12.7)
- moved R14 15.0 mm to (-11.9, 12.7)
- moved TP1 1.00 mm to (5.90, 34.0)
- moved J5 0.93 mm to (-5.13, 38.9)
- moved R4 0.25 mm to (1.25, 20.3)
- moved R5 0.25 mm to (3.15, 20.3)
Connections:
- J2 pad 3: TFT_CLK -> Net-(J2-SCL)
- J2 pad 4: TFT_DC -> Net-(J2-DC)
- J2 pad 6: TFT_MOSI -> Net-(J2-SDA)
Routing:
- net GND: track 145.0 -> 126.0 mm, vias 126 -> 116
- net Net-(J4-PadT): track 22.1 -> 34.2 mm
- net TFT_CLK: track 14.5 -> 2.36 mm, vias 1 -> 0
- net Net-(J2-SCL): track 0.00 -> 11.3 mm, vias 0 -> 1
- net +3.3V: track 264.3 -> 275.3 mm, vias 10 -> 11
- net TFT_MOSI: track 12.4 -> 1.85 mm, vias 1 -> 0
- net TFT_DC: track 11.6 -> 2.06 mm, vias 1 -> 0
- net Net-(J2-DC): track 0.00 -> 8.16 mm, vias 0 -> 1
- net Net-(J2-SDA): track 0.00 -> 7.53 mm, vias 0 -> 1
- net LEVER_SW: track 32.5 -> 39.4 mm, vias 0 -> 2
- net SMPS: track 34.1 -> 29.5 mm
- net Net-(J4-PadR): track 26.0 -> 30.5 mm
- net Net-(R13-Pad2): track 7.92 -> 11.4 mm
- net MOTOR_RIN: track 34.4 -> 37.4 mm
- net AUDIO_SW: track 56.7 -> 59.2 mm
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Other:
- board text added: "V2.0"
- board text removed: "V1.2"
