File: SmaCon.kicad_sch (KiCad schematic)
At the start: 0 parts

Commit message: 回路図作成
Parts:
- added C1, C6: 1uF, symbol Device:C_Small
- added C2, C7: 4.7uF, symbol Device:C_Small
- added C3: 0.1uF, symbol Device:C_Small
- added C4, C5: 10pF, symbol Device:C_Small
- added F1: Polyfuse, symbol Device:Polyfuse_Small
- added J1: GT911, symbol SmaCon:GT911
- added J2: USB_C_Receptacle, symbol SmaCon:USB_C_Receptacle
- added J3: ST7789, symbol SmaCon:ST7789
- added J4: Conn_01x03, symbol Connector_Generic:Conn_01x03
- added J5: STM32_Debug, symbol SmaCon:STM32_Debug_5pin
- added J6: DM3AT-SF-PEJM5, symbol SmaCon:DM3AT-SF-PEJM5
- added J7: AudioJack, symbol Connector:AudioJack3_Switch
- added L1: L, symbol Device:L_Small
- added L2: 2.2uH, symbol Device:L_Small
- added LS1: Speaker, symbol Device:Speaker
- added M1: LD14-002, symbol Motor:Motor_DC
- added Q1: AO3400A, symbol Device:Q_NMOS_GSD
- added R1, R11, R14, R6, R7, R8: 10k, symbol Device:R_Small
- added R10: 4.7k, symbol Device:R_Small
- added R12, R13: 100, symbol Device:R_Small
- added R2: 50, symbol Device:R_Small
- added R3, R4: 5.1k, symbol Device:R_Small
- added R5: 470, symbol Device:R_Small
- added R9: 1M, symbol Device:R_Small
- added RV1: Potentiometer_Dual, symbol Device:R_Potentiometer_Dual_Separate
- added SW1: SW_TMHU27, symbol SmaCon:SW_TMHU27
- added SW2, SW3, SW4, SW5: SW_Push, symbol Switch:SW_Push
- added U1: NJM2884U1, Package_TO_SOT_SMD:SOT-89-5_Handsoldering, symbol SmaCon:NJM2884U1
- added U2: BD45285, symbol SmaCon:BD45285
- added U3: LXES11DAA2-137, symbol SmaCon:LXES11DAA2-137
- added U4: STM32U575CIUxQ, symbol SmaCon:STM32U575CIUxQ
- added U5: YMF825, symbol SmaCon:YMF825
- added U6: BD6211, symbol SmaCon:BD6211
- added Y1: 12.288MHz, symbol Device:Crystal_Small
Connections:
- new net: R10.2, R11.1, SW1.1
- new net: C6.2, U5.10 (VREF)
- new net: C7.1, LS1.2, U5.14 (SPOUT1)
- new net: LS1.1, U5.16 (SPOUT2)
- new net: C4.1, R9.2, U5.23 (XI), Y1.2
- new net: C5.1, R9.1, U5.24 (XO), Y1.1
- new net: Q1.1 (G), R5.2, R6.1
- new net: M1.1 (+), U6.1 (OUT1)
- new net: M1.2 (-), U6.7 (OUT2)
- new net: R11.2, SW1.3 (2)
- new net: J7.R, R12.2
- new net: J7.T, R13.2
- new net: J2.A5 (CC1), R4.1
- new net: F1.2, J2.A4 (VBUS), J2.A9 (VBUS), J2.B4 (VBUS), J2.B9 (VBUS)
- new net: J2.B5 (CC2), R3.1
- new net: C7.2, R12.1, R13.1, R14.1
- new net: J3.10 (LEDA), R2.2
- new net: L2.1, U4.20 (VLXSMPS)
- new net: J3.11 (LEDK), J3.12 (LEDK), J3.13 (LEDK), J3.14 (LEDK), Q1.3 (D)
- new net: F1.1, L1.2
- new net +3.3V: C2.1, J1.6 (VCC), J3.9 (VDD), J5.3 (VDD), J6.4 (VDD), R1.1, R7.1, R8.1, RV1.1, RV1.4, U1.4 (Vout), U2.5 (VDD), U4.1 (VBAT), U4.21 (VDDSMPS), U4.25 (VDD), U4.36 (VDD), U4.48 (VDD), U4.9 (VDDA), U5.8 (VDD), U5.9 (IOVDD)
- new net +5V: C1.1, L1.1, R2.1, U1.1 (CONTROL), U1.5 (Vin), U5.11 (SPVDD), U6.2 (VCC), U6.3 (VCC), U6.6 (VREF)
- new net AUDIO_SW: J7.SN, U4.38 (PA15)
- new net COM_RX: J4.1 (Pin_1), U4.13 (PA3)
- new net COM_TX: J4.3 (Pin_3), U4.12 (PA2)
- new net D+: J2.A6 (D+), J2.B6 (D+), U3.2 (IN2)
- new net D-: J2.A7 (D-), J2.B7 (D-), U3.1 (IN1)
- new net GND: C1.2, C2.2, C3.2, C4.2, C5.2, C6.1, J1.1 (GND), J1.3 (INT), J2.A1 (GND), J2.A12 (GND), J2.B1 (GND), J2.B12 (GND), J3.1 (GND), J3.8 (GND), J4.2 (Pin_2), J5.1 (GND), J6.10 (SW_A), J6.6 (VSS), J7.S, Q1.2 (S), R14.2, R3.2, R4.2, R6.2, RV1.3, RV1.6, SW1.4 (C), SW2.1, SW3.1, SW4.1, SW5.1, U1.2 (GND), U2.1 (ER), U2.2 (SUB), U2.3 (GND), U3.3 (GND), U3.6 (GND), U4.22 (VSSSMPS), U4.24 (VSS), U4.35 (VSS), U4.44 (PH3), U4.47 (VSS), U4.8 (VSSA), U5.12 (SPVSS), U5.18 (VSS), U5.19 (TESTMODE0), U5.20 (TESTMODE1), U5.21 (TESTINA), U5.22 (TESTINB), U6.8 (GND)
- new net LEVER_SW: R10.1, R8.2, SW1.2 (T), U4.14 (PA4)
- new net MOTOR_FIN: U4.31 (PA10), U6.4 (FIN)
- new net MOTOR_RIN: U4.19 (PB1), U6.5 (RIN)
- new net NRST: J5.2 (NRST), U4.7 (NRST)
- new net POS_H: RV1.2, U4.10 (PA0)
- new net POS_V: RV1.5, U4.11 (PA1)
- new net RESET: C3.1, J1.2 (RESET), J3.2 (RESET), R1.2, U2.4 (Vout), U5.7 (RST_N)
- new net SD_CLK: J6.5 (CLK), U4.39 (PB3)
- new net SD_CS: J6.2 (CD_DAT3), U4.45 (PB8)
- new net SD_MISO: J6.7 (DAT0), R7.2, U4.40 (PB4)
- new net SD_MOSI: J6.3 (CMD), U4.41 (PB5)
- new net SD_SW: J6.9 (SW_B), U4.2 (PC13)
- new net SMPS: L2.2, U4.23 (VDD11), U4.46 (VDD11)
- new net SOUND_CLK: U4.26 (PB13), U5.5 (SCK)
- new net SOUND_CS: U4.29 (PA8), U5.6 (SS_N)
- new net SOUND_MISO: U4.27 (PB14), U5.3 (SO)
- new net SOUND_MOSI: U4.28 (PB15), U5.4 (SI)
- new net SWCLK: J5.4 (SWCLK), U4.37 (PA14)
- new net SWDIO: J5.5 (SWDIO), U4.34 (PA13)
- new net SW_A: SW2.2, U4.3 (PC14)
- new net SW_B: SW3.2, U4.4 (PC15)
- new net SW_C: SW4.2, U4.5 (PH0)
- new net SW_D: SW5.2, U4.6 (PH1)
- new net TFT_CLK: J3.3 (SCL), U4.15 (PA5)
- new net TFT_CS: J3.5 (CS), U4.30 (PA9)
- new net TFT_DC: J3.4 (DC), U4.16 (PA6)
- new net TFT_LED: R5.1, U4.18 (PB0)
- new net TFT_MOSI: J3.6 (SDA), U4.17 (PA7)
- new net TOUCH_SCL: J1.5 (SCL), U4.42 (PB6)
- new net TOUCH_SDA: J1.4 (SDA), U4.43 (PB7)
- new net USB_DM: U3.5 (OUT1), U4.32 (PA11)
- new net USB_DP: U3.4 (OUT2), U4.33 (PA12)
- no-connect marks 0 -> 8
Other:
- note added: "5V -> 3.3V"
- note added: "Controller"
- note added: "FM Sound Generator"
- note added: "Lever SW"
- note added: "Micro SD"
- note added: "Reset IC"
- note added: "TFT 2.8inch"
- note added: "Touch Pad"
- note added: "Vibration Motor"

Commit message: EEPROMに変更、マイコン型番変更
Parts:
- removed J6: DM3AT-SF-PEJM5, symbol SmaCon:DM3AT-SF-PEJM5
- added U1: 25LC080C, symbol SmaCon:25LC080C
- renumbered C6 to C4, C7 to C5, C4 to C6, C5 to C7, J2 to J1, J5 to J2, J4 to J3, J1 to J4, J3 to J5, J7 to J6, R7 to R1, R9 to R10, R6 to R11, R2 to R12, R12 to R13, R13 to R14, R3 to R2, R4 to R3, R8 to R4, R10 to R5, R11 to R6, R1 to R7, R5 to R8, R14 to R9, SW2 to SW1, SW3 to SW2, SW4 to SW3, SW5 to SW4, SW1 to SW5, U3 to U2, U1 to U3, U6 to U4, U4 to U5, U2 to U6, U5 to U7
Connections:
- net +3.3V: now also U1.8 (VCC)
- net GND: now also U1.4 (GND)
- net SD_CLK renamed EEPROM_CLK
- net EEPROM_CLK: now also U1.6 (SCK)
- net SD_CS renamed EEPROM_CS
- net EEPROM_CS: now also U1.1 (~{CS})
- net SD_MISO: no longer names the net of R1.2
- net SD_MISO: now also U1.3 (~{WP}); no longer U5.40 (PB4)
- net SD_MOSI renamed EEPROM_MOSI
- net EEPROM_MOSI: now also U1.5 (MOSI)
- net SD_SW renamed EEPROM_HOLD
- net EEPROM_HOLD: now also U1.7 (~{HOLD})
- new net EEPROM_MISO: U1.2 (MISO), U5.40 (PB4)
- no-connect marks 8 -> 6
Other:
- note added: "EEPROM"
- note removed: "Micro SD"
- moved on the sheet: R1

Commit message: 部品選定
Parts:
- removed J3: Conn_01x03, symbol Connector_Generic:Conn_01x03
- added C10, C9: 2.2uF, SmaCon:1005Metric, symbol Device:C_Small
- added C11, C6, C7, C8: 0.1uF, SmaCon:1005Metric, symbol Device:C_Small
- added C12, C17, C3, C5: 10uF, SmaCon:1608Metric, symbol Device:C_Small
- added J6: Conn_01x04, SmaCon:PinHeader_1x04_P2.54mm_Horizontal, symbol Connector_Generic:Conn_01x04
- added R7: 100, SmaCon:2012Metric, symbol Device:R_Small
- C1: value 1uF -> 2.2uF; footprint (none) -> SmaCon:1005Metric
- C13: renamed from C4; footprint (none) -> SmaCon:1005Metric
- C14: renamed from C5; footprint (none) -> SmaCon:1608Metric
- C15: renamed from C6; footprint (none) -> SmaCon:1005Metric
- C16: renamed from C7; footprint (none) -> SmaCon:1005Metric
- C2: value 4.7uF -> 2.2uF; footprint (none) -> SmaCon:1005Metric
- C4: renamed from C3; footprint (none) -> SmaCon:1005Metric
- F1: footprint (none) -> SmaCon:3216Metric
- J1: footprint (none) -> SmaCon:USB Type-C 5077CR-16SMC2-BK-TR
- J2: renamed from J5; footprint (none) -> SmaCon:Hirose_FH12-18S-0.5SH_1x18-1MP_P0.50mm_Horizontal
- J3: renamed from J4; footprint (none) -> SmaCon:Hirose_FH12-6S-0.5SH_1x06-1MP_P0.50mm_Horizontal
- J4: renamed from J6; footprint (none) -> SmaCon:PJ-3420
- J5: renamed from J2; footprint (none) -> SmaCon:STM32_Debug_5pin
- L1: footprint (none) -> SmaCon:1608Metric
- L2: footprint (none) -> SmaCon:2012Metric
- LS1: footprint (none) -> SmaCon:micro_speaker
- M1: footprint (none) -> SmaCon:LD14-002
- Q1: footprint (none) -> SmaCon:SOT-23
- R1: renamed from R2; footprint (none) -> SmaCon:1005Metric
- R10: renamed from R13; footprint (none) -> SmaCon:2012Metric
- R11: renamed from R14; footprint (none) -> SmaCon:2012Metric
- R12: renamed from R4; footprint (none) -> SmaCon:1005Metric
- R13: renamed from R5; footprint (none) -> SmaCon:1005Metric
- R14: renamed from R6; footprint (none) -> SmaCon:1005Metric
- R15: renamed from R1; footprint (none) -> SmaCon:1005Metric
- R2: renamed from R3; footprint (none) -> SmaCon:1005Metric
- R3: renamed from R7; footprint (none) -> SmaCon:1005Metric
- R4: renamed from R8; footprint (none) -> SmaCon:1005Metric
- R5: renamed from R11; footprint (none) -> SmaCon:1005Metric
- R6: renamed from R12; value 50 -> 100; footprint (none) -> SmaCon:2012Metric
- R8: renamed from R9; footprint (none) -> SmaCon:1005Metric
- R9: renamed from R10; footprint (none) -> SmaCon:1005Metric
- RV1: footprint (none) -> SmaCon:JT8P-3.2T-B10K-1-16Y
- SW1, SW2, SW3, SW4: footprint (none) -> SmaCon:tact_switch
- SW5: footprint (none) -> SmaCon:SW_TMHU27
- U1: renamed from U2; footprint (none) -> SmaCon:LXES11D
- U2: renamed from U3; footprint Package_TO_SOT_SMD:SOT-89-5_Handsoldering -> SmaCon:SOT-89-5
- U3: renamed from U6; footprint (none) -> SmaCon:SOT-23-5
- U4: renamed from U5; footprint (none) -> SmaCon:QFN-48-1EP_7x7mm_P0.5mm_EP5.3x5.3mm
- U5: renamed from U7; footprint (none) -> SmaCon:SSOP-24_5.3x8.2mm_P0.65mm
- U6: renamed from U1; footprint (none) -> SmaCon:MSOP-8_3x3mm_P0.65mm
- U7: renamed from U4; footprint (none) -> SmaCon:SOP-8_4.4x5.0mm_P1.27mm
- Y1: footprint (none) -> SmaCon:Crystal_SMD_TXC_AX_8045-2Pin_8.0x4.5mm
Connections:
- net +3.3V: now also C11.1, C3.1, C6.1, C7.1, C8.1, J6.2 (Pin_2)
- net +5V: now also C12.1, C17.1, C5.1, R7.1
- net COM_RX: now also J6.4 (Pin_4)
- net COM_TX: now also J6.3 (Pin_3)
- net GND: now also C10.2, C11.2, C12.2, C17.2, C3.2, C5.2, C6.2, C7.2, C8.2, C9.2, J6.1 (Pin_1)
- net SMPS: now also C10.1, C9.1
- net at J2.10 (LEDA), R6.2: now also R7.2
Other:
- note added: "Debug port"
- note added: "Extension port"
- note added: "MCU"
- note added: "USB"
- moved on the sheet: C1, C13, C14, C15, C16, C2, C4, F1, J1, J2, J3, J4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

Commit message: 基板 V1.0
Parts:
- added TP1: TestPoint, SmaCon:TestPoint_THTPad_D1.2mm_Drill0.8mm, symbol Connector:TestPoint
- J4: symbol Connector:AudioJack3_Switch -> Connector_Audio:AudioJack3_Switch
Connections:
- net NRST is gone; now on net RESET: J5.2 (NRST), U4.7 (NRST)
- net D+: now also U1.1 (IN1); no longer U1.2 (IN2)
- net D-: now also U1.2 (IN2); no longer U1.1 (IN1)
- net at R15.2, U6.3 (~{WP}): now also U6.7 (~{HOLD})
- net EEPROM_HOLD renamed TEST
- net TEST: now also TP1.1; no longer U6.7 (~{HOLD})
Other:
- moved on the sheet: U1
Changed lines of the file:
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@@
   (title_block
     (title "SmaCon")
-    (date "2023-02-12")
+    (date "2023-07-24")
     (rev "V1.0")
     (company "https://github.com/KimiakiK")
   )
+  (junction (at 236.22 229.87) (diameter 0) (color 0 0 0 0)
+  )
   (junction (at 219.71 171.45) (diameter 0) (color 0 0 0 0)
   )
@@
   (junction (at 88.9 179.07) (diameter 0) (color 0 0 0 0)
   )
-  (junction (at 102.87 67.31) (diameter 0) (color 0 0 0 0)
+  (junction (at 102.87 69.85) (diameter 0) (color 0 0 0 0)
   )
   (junction (at 224.79 49.53) (diameter 0) (color 0 0 0 0)
@@
     (stroke (width 0) (type default))
   )
-  (wire (pts (xy 81.28 57.15) (xy 91.44 57.15))
-    (stroke (width 0) (type default))
-  )
   (wire (pts (xy 325.12 60.96) (xy 325.12 62.23))
     (stroke (width 0) (type default))
@@
     (stroke (width 0) (type default))
   )
-  (wire (pts (xy 101.6 67.31) (xy 102.87 67.31))
+  (wire (pts (xy 101.6 69.85) (xy 102.87 69.85))
     (stroke (width 0) (type default))
   )
@@
     (stroke (width 0) (type default))
   )
-  (wire (pts (xy 102.87 67.31) (xy 104.14 67.31))
+  (wire (pts (xy 102.87 69.85) (xy 104.14 69.85))
     (stroke (width 0) (type default))
   )
@@
     (stroke (width 0) (type default))
   )
+  (wire (pts (xy 236.22 232.41) (xy 236.22 229.87))
+    (stroke (width 0) (type default))
+  )
   (wire (pts (xy 187.96 227.33) (xy 187.96 236.22))
     (stroke (width 0) (type default))
@@
     (stroke (width 0) (type default))
   )
+  (wire (pts (xy 90.17 57.15) (xy 81.28 57.15))
+    (stroke (width 0) (type default))
+  )
+  (wire (pts (xy 175.26 133.35) (xy 182.88 133.35))
+    (stroke (width 0) (type default))
+  )
   (wire (pts (xy 302.26 158.75) (xy 320.04 158.75))
     (stroke (width 0) (type default))
@@
     (stroke (width 0) (type default))
   )
+  (wire (pts (xy 237.49 232.41) (xy 236.22 232.41))
+    (stroke (width 0) (type default))
+  )
   (wire (pts (xy 48.26 184.15) (xy 48.26 187.96))
     (stroke (width 0) (type default))
@@
     (stroke (width 0) (type default))
   )
+  (wire (pts (xy 90.17 62.23) (xy 90.17 57.15))
+    (stroke (width 0) (type default))
+  )
   (wire (pts (xy 328.93 58.42) (xy 328.93 62.23))
     (stroke (width 0) (type default))
@@
     (stroke (width 0) (type default))
   )
+  (wire (pts (xy 91.44 62.23) (xy 90.17 62.23))
+    (stroke (width 0) (type default))
+  )
   (wire (pts (xy 342.9 143.51) (xy 350.52 143.51))
     (stroke (width 0) (type default))
@@
     (effects (font (size 1.27 1.27)) (justify left bottom))
   )
+  (label "TEST" (at 177.8 133.35 0) (fields_autoplaced)
+    (effects (font (size 1.27 1.27)) (justify left bottom))
+  )
   (global_label "POS_V" (shape input) (at 182.88 156.21 180) (fields_autoplaced)
     (effects (font (size 1.27 1.27)) (justify right))
@@
     )
   )
+  (global_label "RESET" (shape input) (at 143.51 231.14 0) (fields_autoplaced)
+    (effects (font (size 1.27 1.27)) (justify left))
+    (property "Intersheetrefs" "${INTERSHEET_REFS}" (at 151.6683 231.0606 0)
+      (effects (font (size 1.27 1.27)) (justify left) hide)
+    )
+  )
   (global_label "SOUND_CS" (shape input) (at 320.04 153.67 180) (fields_autoplaced)
     (effects (font (size 1.27 1.27)) (justify right))
@@
     )
   )
+  (global_label "RESET" (shape input) (at 182.88 146.05 180) (fields_autoplaced)
+    (effects (font (size 1.27 1.27)) (justify right))
+    (property "Intersheetrefs" "${INTERSHEET_REFS}" (at 174.1497 146.05 0)
+      (effects (font (size 1.27 1.27)) (justify right) hide)
+    )
+  )
   (global_label "SOUND_MOSI" (shape input) (at 228.6 151.13 0) (fields_autoplaced)
     (effects (font (size 1.27 1.27)) (justify left))
@@
     )
   )
-  (global_label "USB_DM" (shape input) (at 114.3 57.15 0) (fields_autoplaced)
-    (effects (font (size 1.27 1.27)) (justify left))
-    (property "Intersheetrefs" "${INTERSHEET_REFS}" (at 124.2121 57.0706 0)
-      (effects (font (size 1.27 1.27)) (justify left) hide)
-    )
-  )
-  (global_label "NRST" (shape input) (at 143.51 231.14 0) (fields_autoplaced)
+  (global_label "USB_DM" (shape input) (at 114.3 59.69 0) (fields_autoplaced)
     (effects (font (size 1.27 1.27)) (justify left))
-    (property "Intersheetrefs" "${INTERSHEET_REFS}" (at 150.7007 231.0606 0)
+    (property "Intersheetrefs" "${INTERSHEET_REFS}" (at 124.2121 59.6106 0)
       (effects (font (size 1.27 1.27)) (justify left) hide)
     )
@@
     )
   )
-  (global_label "EEPROM_HOLD" (shape input) (at 237.49 232.41 180) (fields_autoplaced)
-    (effects (font (size 1.27 1.27)) (justify right))
-    (property "Intersheetrefs" "${INTERSHEET_REFS}" (at 221.0376 232.41 0)
-      (effects (font (size 1.27 1.27)) (justify right) hide)
-    )
-  )
   (global_label "MOTOR_RIN" (shape input) (at 340.36 238.76 0) (fields_autoplaced)
     (effects (font (size 1.27 1.27)) (justify left))
@@
     )
   )
-  (global_label "USB_DP" (shape input) (at 114.3 59.69 0) (fields_autoplaced)
+  (global_label "USB_DP" (shape input) (at 114.3 62.23 0) (fields_autoplaced)
     (effects (font (size 1.27 1.27)) (justify left))
-    (property "Intersheetrefs" "${INTERSHEET_REFS}" (at 124.0307 59.6106 0)
+    (property "Intersheetrefs" "${INTERSHEET_REFS}" (at 124.0307 62.1506 0)
       (effects (font (size 1.27 1.27)) (justify left) hide)
     )
@@
     )
   )
-  (global_label "NRST" (shape input) (at 182.88 146.05 180) (fields_autoplaced)
-    (effects (font (size 1.27 1.27)) (justify right))
-    (property "Intersheetrefs" "${INTERSHEET_REFS}" (at 175.6893 146.1294 0)
-      (effects (font (size 1.27 1.27)) (justify right) hide)
-    )
-  )
   (global_label "EEPROM_MISO" (shape input) (at 212.09 121.92 90) (fields_autoplaced)
     (effects (font (size 1.27 1.27)) (justify left))
@@
     )
   )
-  (global_label "EEPROM_HOLD" (shape input) (at 182.88 133.35 180) (fields_autoplaced)
-    (effects (font (size 1.27 1.27)) (justify right))
-    (property "Intersheetrefs" "${INTERSHEET_REFS}" (at 166.4276 133.35 0)
-      (effects (font (size 1.27 1.27)) (justify right) hide)
-    )
-  )
   (symbol (lib_id "Device:R_Small") (at 69.85 228.6 0) (unit 1)
     (in_bom yes) (on_board yes) (dnp no)
@@
     )
   )
+  (symbol (lib_id "Connector:TestPoint") (at 175.26 133.35 0) (unit 1)
+    (in_bom yes) (on_board yes) (dnp no)
+    (property "Reference" "TP1" (at 175.26 128.27 0)
+      (effects (font (size 1.27 1.27)))
+    )
+    (property "Value" "TestPoint" (at 165.1 132.08 0)
+      (effects (font (size 1.27 1.27)) (justify left) hide)
+    )
+    (property "Footprint" "SmaCon:TestPoint_THTPad_D1.2mm_Drill0.8mm" (at 180.34 133.35 0)
+      (effects (font (size 1.27 1.27)) hide)
+    )
+    (property "Datasheet" "~" (at 180.34 133.35 0)
+      (effects (font (size 1.27 1.27)) hide)
+    )
+    (pin "1")
+    (instances
+      (project "SmaCon"
+        (path "/0ddb81ff-5188-45bf-8749-168d9d994e1f"
+          (reference "TP1") (unit 1)
+        )
+      )
+    )
+  )
   (symbol (lib_id "Device:R_Small") (at 69.85 233.68 0) (unit 1)
     (in_bom yes) (on_board yes) (dnp no)
@@
     )
   )
-  (symbol (lib_id "Connector:AudioJack3_Switch") (at 373.38 165.1 0) (mirror y) (unit 1)
+  (symbol (lib_id "Connector_Audio:AudioJack3_Switch") (at 373.38 165.1 0) (mirror y) (unit 1)
     (in_bom yes) (on_board yes) (dnp no)
     (property "Reference" "J4" (at 370.84 154.94 0)
@@
     )
   )
-  (symbol (lib_id "power:GND") (at 102.87 67.31 0) (unit 1)
+  (symbol (lib_id "power:GND") (at 102.87 69.85 0) (unit 1)
     (in_bom yes) (on_board yes) (dnp no)
-    (property "Reference" "#PWR04" (at 102.87 73.66 0)
+    (property "Reference" "#PWR04" (at 102.87 76.2 0)
       (effects (font (size 1.27 1.27)) hide)
     )
-    (property "Value" "GND" (at 102.87 71.12 0)
+    (property "Value" "GND" (at 102.87 73.66 0)
       (effects (font (size 1.27 1.27)))
     )
-    (property "Footprint" "" (at 102.87 67.31 0)
+    (property "Footprint" "" (at 102.87 69.85 0)
       (effects (font (size 1.27 1.27)) hide)
     )
-    (property "Datasheet" "" (at 102.87 67.31 0)
+    (property "Datasheet" "" (at 102.87 69.85 0)
       (effects (font (size 1.27 1.27)) hide)
     )
@@
     )
   )
-  (symbol (lib_id "SmaCon:LXES11DAA2-137") (at 102.87 58.42 0) (unit 1)
+  (symbol (lib_id "SmaCon:LXES11DAA2-137") (at 102.87 60.96 0) (unit 1)
     (in_bom yes) (on_board yes) (dnp no)
-    (property "Reference" "U1" (at 102.87 48.26 0)
+    (property "Reference" "U1" (at 102.87 50.8 0)
       (effects (font (size 1.27 1.27)))
     )
-    (property "Value" "LXES11DAA2-137" (at 102.87 50.8 0)
+    (property "Value" "LXES11DAA2-137" (at 102.87 53.34 0)
       (effects (font (size 1.27 1.27)))
     )
-    (property "Footprint" "SmaCon:LXES11D" (at 102.87 58.42 0)
+    (property "Footprint" "SmaCon:LXES11D" (at 102.87 60.96 0)
       (effects (font (size 1.27 1.27)) hide)
     )
-    (property "Datasheet" "" (at 102.87 58.42 0)
+    (property "Datasheet" "" (at 102.87 60.96 0)
       (effects (font (size 1.27 1.27)) hide)
     )

Commit message: 基板 V1.1
Connections:
- net POS_H: now also RV1.5; no longer RV1.2
- net POS_V: now also RV1.2; no longer RV1.5
Changed lines of the file:
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@@
   (title_block
     (title "SmaCon")
-    (date "2023-07-24")
-    (rev "V1.0")
+    (date "2023-08-05")
+    (rev "V1.1")
     (company "https://github.com/KimiakiK")
   )
@@
     )
   )
-  (global_label "POS_H" (shape input) (at 57.15 177.8 0) (fields_autoplaced)
-    (effects (font (size 1.27 1.27)) (justify left))
-    (property "Intersheetrefs" "${INTERSHEET_REFS}" (at 65.6712 177.7206 0)
+  (global_label "POS_H" (shape input) (at 74.93 181.61 0) (fields_autoplaced)
+    (effects (font (size 1.27 1.27)) (justify left))
+    (property "Intersheetrefs" "${INTERSHEET_REFS}" (at 83.4512 181.5306 0)
       (effects (font (size 1.27 1.27)) (justify left) hide)
     )
@@
     )
   )
-  (global_label "POS_V" (shape input) (at 74.93 181.61 0) (fields_autoplaced)
-    (effects (font (size 1.27 1.27)) (justify left))
-    (property "Intersheetrefs" "${INTERSHEET_REFS}" (at 83.2093 181.5306 0)
-      (effects (font (size 1.27 1.27)) (justify left) hide)
-    )
+  (global_label "POS_V" (shape input) (at 57.15 177.8 0) (fields_autoplaced)
+    (effects (font (size 1.27 1.27)) (justify left))
+    (property "Intersheetrefs" "${INTERSHEET_REFS}" (at 65.4293 177.7206 0)
+      (effects (font (size 1.27 1.27)) (justify left) hide)
+    )
